File: pcb/ghost.kicad_pcb (KiCad board)
At the start: 2 copper layers, 56.6 x 64.3 mm, 15 parts, among them SW1 SW_SPDT, U1 ATtiny85-20S

Commit message: altera resistores dos leds
Parts:
- R1, R2: value 2k2 -> 47R
Changed lines of the file:
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@@
       (effects (font (size 1 1) (thickness 0.15)) (justify mirror))
     )
-    (fp_text value "2k2" (at 0 -1.43) (layer "B.Fab")
+    (fp_text value "47R" (at 0 -1.43) (layer "B.Fab")
       (effects (font (size 1 1) (thickness 0.15)) (justify mirror))
     )
@@
       (effects (font (size 1 1) (thickness 0.15)) (justify mirror))
     )
-    (fp_text value "2k2" (at 0 -1.43) (layer "B.Fab")
+    (fp_text value "47R" (at 0 -1.43) (layer "B.Fab")
       (effects (font (size 1 1) (thickness 0.15)) (justify mirror))
     )
