File: pcb/ghost.kicad_sch (KiCad schematic)
At the start: 14 parts, among them SW1 SW_SPDT, U1 ATtiny85-20S

Commit message: altera resistores dos leds
Parts:
- R1, R2: value 2k2 -> 47R
Changed lines of the file:
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@@
       (effects (font (size 1.27 1.27)) (justify left))
     )
-    (property "Value" "2k2" (id 1) (at 198.12 74.9299 0)
+    (property "Value" "47R" (id 1) (at 198.12 74.9299 0)
       (effects (font (size 1.27 1.27)) (justify left))
     )
@@
       (effects (font (size 1.27 1.27)) (justify left))
     )
-    (property "Value" "2k2" (id 1) (at 186.69 74.9299 0)
+    (property "Value" "47R" (id 1) (at 186.69 74.9299 0)
       (effects (font (size 1.27 1.27)) (justify left))
     )
@@
     )
     (path "/c09425c9-49cf-4a9c-9231-e239993b348c"
-      (reference "R1") (unit 1) (value "2k2") (footprint "Resistor_SMD:R_0603_1608Metric")
+      (reference "R1") (unit 1) (value "47R") (footprint "Resistor_SMD:R_0603_1608Metric")
     )
     (path "/0219e57b-4b68-4a94-85b0-1f597adf6c7b"
-      (reference "R2") (unit 1) (value "2k2") (footprint "Resistor_SMD:R_0603_1608Metric")
+      (reference "R2") (unit 1) (value "47R") (footprint "Resistor_SMD:R_0603_1608Metric")
     )
     (path "/ff0630d9-e2cb-4ed4-87a6-9699c2ef85a8"
